File: Controller/controller_board/controller_board.kicad_pcb (KiCad board)
At the start: 2 copper layers, 97.8 x 109.7 mm, 50 parts, among them J1 Conn_02x06_Odd_Even, J10 Conn_Knob_LED, J11 Conn_IP_LED, J12 Conn_Cloud_ERR, J13 Conn_Network_ERR, J14 Conn_MQTT_ERR, J15 Conn_Knob, J2 Conn_02x03_Counter_Clockwise, J3 Conn_02x03_Counter_Clockwise, J4 Conn_BATTERY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

Commit message: add stl files
Parts:
- J10: value Conn_Knob_LED -> Conn_IP_LED
- J11: value Conn_IP_LED -> Conn_Net_ERR
- J12: value Conn_Cloud_ERR -> Conn_Knob_LED
- J13: value Conn_Network_ERR -> Conn_Peri_ERR
- J14: value Conn_MQTT_ERR -> Conn_SP_LED
- J9: value Conn_SP_LED -> Conn_MQTT_ERR
- R1, R2, R21, R22, R3, R4: value R -> 10k
- R10, R11, R12, R13, R14, R16, R20, R5, R6, R7, R8, R9: value R -> 680R
- R15, R17, R18, R19: value R -> 220R
- R23: value R -> 1k
- R24: value R -> 3.3k
- R25, R26: value R -> 4.7k
Changed lines of the file:
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@@
       (effects (font (size 1 1) (thickness 0.15)))
     )
-    (fp_text value R (at 5.08 2.37) (layer F.Fab)
+    (fp_text value 4.7k (at 5.08 2.37) (layer F.Fab)
       (effects (font (size 1 1) (thickness 0.15)))
     )
@@
       (effects (font (size 1 1) (thickness 0.15)))
     )
-    (fp_text value R (at 5.08 2.37) (layer F.Fab)
+    (fp_text value 4.7k (at 5.08 2.37) (layer F.Fab)
       (effects (font (size 1 1) (thickness 0.15)))
     )
@@
       (effects (font (size 1 1) (thickness 0.15)))
     )
-    (fp_text value R (at 5.08 2.37 90) (layer F.Fab)
+    (fp_text value 3.3k (at 5.08 2.37 90) (layer F.Fab)
       (effects (font (size 1 1) (thickness 0.15)))
     )
@@
       (effects (font (size 1 1) (thickness 0.15)))
     )
-    (fp_text value R (at 5.08 2.37 90) (layer F.Fab)
+    (fp_text value 1k (at 5.08 2.37 90) (layer F.Fab)
       (effects (font (size 1 1) (thickness 0.15)))
     )
@@
       (effects (font (size 1 1) (thickness 0.15)))
     )
-    (fp_text value Conn_MQTT_ERR (at 0 4.87) (layer F.Fab)
+    (fp_text value Conn_SP_LED (at 0 4.87) (layer F.Fab)
       (effects (font (size 1 1) (thickness 0.15)))
     )
@@
       (effects (font (size 1 1) (thickness 0.15)))
     )
-    (fp_text value Conn_Network_ERR (at 0 4.87) (layer F.Fab)
+    (fp_text value Conn_Peri_ERR (at 0 4.87) (layer F.Fab)
       (effects (font (size 1 1) (thickness 0.15)))
     )
@@
       (effects (font (size 1 1) (thickness 0.15)))
     )
-    (fp_text value Conn_Cloud_ERR (at 0 4.87) (layer F.Fab)
+    (fp_text value Conn_Knob_LED (at 0 4.87) (layer F.Fab)
       (effects (font (size 1 1) (thickness 0.15)))
     )
@@
       (effects (font (size 1 1) (thickness 0.15)))
     )
-    (fp_text value Conn_IP_LED (at 0 4.87) (layer F.Fab)
+    (fp_text value Conn_Net_ERR (at 0 4.87) (layer F.Fab)
       (effects (font (size 1 1) (thickness 0.15)))
     )
@@
       (effects (font (size 1 1) (thickness 0.15)))
     )
-    (fp_text value Conn_Knob_LED (at 0 4.87) (layer F.Fab)
+    (fp_text value Conn_IP_LED (at 0 4.87) (layer F.Fab)
       (effects (font (size 1 1) (thickness 0.15)))
     )
@@
       (effects (font (size 1 1) (thickness 0.15)))
     )
-    (fp_text value Conn_SP_LED (at 0 4.87) (layer F.Fab)
+    (fp_text value Conn_MQTT_ERR (at 0 4.87) (layer F.Fab)
       (effects (font (size 1 1) (thickness 0.15)))
     )
@@
       (effects (font (size 1 1) (thickness 0.15)))
     )
-    (fp_text value R (at 5.08 2.37) (layer F.Fab)
+    (fp_text value 10k (at 5.08 2.37) (layer F.Fab)
       (effects (font (size 1 1) (thickness 0.15)))
     )
@@
       (effects (font (size 1 1) (thickness 0.15)))
     )
-    (fp_text value R (at 5.08 2.37) (layer F.Fab)
+    (fp_text value 10k (at 5.08 2.37) (layer F.Fab)
       (effects (font (size 1 1) (thickness 0.15)))
     )
@@
       (effects (font (size 1 1) (thickness 0.15)))
     )
-    (fp_text value R (at 5.08 2.37 90) (layer F.Fab)
+    (fp_text value 680R (at 5.08 2.37 90) (layer F.Fab)
       (effects (font (size 1 1) (thickness 0.15)))
     )
@@
       (effects (font (size 1 1) (thickness 0.15)))
     )
-    (fp_text value R (at 5.08 2.37 90) (layer F.Fab)
+    (fp_text value 220R (at 5.08 2.37 90) (layer F.Fab)
       (effects (font (size 1 1) (thickness 0.15)))
     )
@@
       (effects (font (size 1 1) (thickness 0.15)))
     )
-    (fp_text value R (at 5.08 2.37 90) (layer F.Fab)
+    (fp_text value 220R (at 5.08 2.37 90) (layer F.Fab)
       (effects (font (size 1 1) (thickness 0.15)))
     )
@@
       (effects (font (size 1 1) (thickness 0.15)))
     )
-    (fp_text value R (at 5.08 2.37 90) (layer F.Fab)
+    (fp_text value 220R (at 5.08 2.37 90) (layer F.Fab)
       (effects (font (size 1 1) (thickness 0.15)))
     )
@@
       (effects (font (size 1 1) (thickness 0.15)))
     )
-    (fp_text value R (at 5.08 2.37 90) (layer F.Fab)
+    (fp_text value 680R (at 5.08 2.37 90) (layer F.Fab)
       (effects (font (size 1 1) (thickness 0.15)))
     )
@@
       (effects (font (size 1 1) (thickness 0.15)))
     )
-    (fp_text value R (at 5.08 2.37 90) (layer F.Fab)
+    (fp_text value 220R (at 5.08 2.37 90) (layer F.Fab)
       (effects (font (size 1 1) (thickness 0.15)))
     )
@@
       (effects (font (size 1 1) (thickness 0.15)))
     )
-    (fp_text value R (at 5.08 2.37 90) (layer F.Fab)
+    (fp_text value 680R (at 5.08 2.37 90) (layer F.Fab)
       (effects (font (size 1 1) (thickness 0.15)))
     )
@@
       (effects (font (size 1 1) (thickness 0.15)))
     )
-    (fp_text value R (at 5.08 2.37 90) (layer F.Fab)
+    (fp_text value 680R (at 5.08 2.37 90) (layer F.Fab)
       (effects (font (size 1 1) (thickness 0.15)))
     )
@@
       (effects (font (size 1 1) (thickness 0.15)))
     )
-    (fp_text value R (at 5.08 2.37 90) (layer F.Fab)
+    (fp_text value 680R (at 5.08 2.37 90) (layer F.Fab)
       (effects (font (size 1 1) (thickness 0.15)))
     )
@@
       (effects (font (size 1 1) (thickness 0.15)))
     )
-    (fp_text value R (at 5.08 2.37 90) (layer F.Fab)
+    (fp_text value 680R (at 5.08 2.37 90) (layer F.Fab)
       (effects (font (size 1 1) (thickness 0.15)))
     )
@@
       (effects (font (size 1 1) (thickness 0.15)))
     )
-    (fp_text value R (at 5.08 2.37 90) (layer F.Fab)
+    (fp_text value 680R (at 5.08 2.37 90) (layer F.Fab)
       (effects (font (size 1 1) (thickness 0.15)))
     )
@@
       (effects (font (size 1 1) (thickness 0.15)))
     )
-    (fp_text value R (at 5.08 2.37 90) (layer F.Fab)
+    (fp_text value 680R (at 5.08 2.37 90) (layer F.Fab)
       (effects (font (size 1 1) (thickness 0.15)))
     )
@@
       (effects (font (size 1 1) (thickness 0.15)))
     )
-    (fp_text value R (at 5.08 2.37 90) (layer F.Fab)
+    (fp_text value 680R (at 5.08 2.37 90) (layer F.Fab)
       (effects (font (size 1 1) (thickness 0.15)))
     )
@@
       (effects (font (size 1 1) (thickness 0.15)))
     )
-    (fp_text value R (at 5.08 2.37 90) (layer F.Fab)
+    (fp_text value 680R (at 5.08 2.37 90) (layer F.Fab)
       (effects (font (size 1 1) (thickness 0.15)))
     )
@@
       (effects (font (size 1 1) (thickness 0.15)))
     )
-    (fp_text value R (at 5.08 2.37 90) (layer F.Fab)
+    (fp_text value 680R (at 5.08 2.37 90) (layer F.Fab)
       (effects (font (size 1 1) (thickness 0.15)))
     )
@@
       (effects (font (size 1 1) (thickness 0.15)))
     )
-    (fp_text value R (at 5.08 2.37 90) (layer F.Fab)
+    (fp_text value 680R (at 5.08 2.37 90) (layer F.Fab)
       (effects (font (size 1 1) (thickness 0.15)))
     )
@@
       (effects (font (size 1 1) (thickness 0.15)))
     )
-    (fp_text value R (at 5.08 2.37) (layer F.Fab)
+    (fp_text value 10k (at 5.08 2.37) (layer F.Fab)
       (effects (font (size 1 1) (thickness 0.15)))
     )
@@
       (effects (font (size 1 1) (thickness 0.15)))
     )
-    (fp_text value R (at 5.08 2.37) (layer F.Fab)
+    (fp_text value 10k (at 5.08 2.37) (layer F.Fab)
       (effects (font (size 1 1) (thickness 0.15)))
     )
@@
       (effects (font (size 1 1) (thickness 0.15)))
     )
-    (fp_text value R (at 5.08 2.37) (layer F.Fab)
+    (fp_text value 10k (at 5.08 2.37) (layer F.Fab)
       (effects (font (size 1 1) (thickness 0.15)))
     )
@@
       (effects (font (size 1 1) (thickness 0.15)))
     )
-    (fp_text value R (at 5.08 2.37) (layer F.Fab)
-      (effects (font (size 1 1) (thickness 0.15)))
-    )
+    (fp_text value 10k (at 5.08 2.37) (layer F.Fab)
+      (effects (font (size 1 1) (thickness 0.15)))
+    )
