File: Controller/controller_board/controller_board.sch (KiCad schematic (older format))
At the start: 47 parts, among them J1 Conn_02x06_Odd_Even, J10 Conn_Knob_LED, J11 Conn_IP_LED, J12 Conn_Cloud_ERR, J13 Conn_Network_ERR, J14 Conn_MQTT_ERR, J15 Conn_Knob, J2 Conn_02x03_Counter_Clockwise, J3 Conn_02x03_Counter_Clockwise, J4 Conn_BATTERY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

Commit message: add stl files
Parts:
- J10: value Conn_Knob_LED -> Conn_IP_LED
- J11: value Conn_IP_LED -> Conn_Net_ERR
- J12: value Conn_Cloud_ERR -> Conn_Knob_LED
- J13: value Conn_Network_ERR -> Conn_Peri_ERR
- J14: value Conn_MQTT_ERR -> Conn_SP_LED
- J9: value Conn_SP_LED -> Conn_MQTT_ERR
- R1, R2, R21, R22, R3, R4: value R -> 10k
- R10, R11, R12, R13, R14, R16, R20, R5, R6, R7, R8, R9: value R -> 680R
- R15, R17, R18, R19: value R -> 220R
- R23: value R -> 1k
- R24: value R -> 3.3k
- R25, R26: value R -> 4.7k
Changed lines of the file:
@@
 P 2000 4400
 F 0 "R3" V 2100 4350 50  0000 C CNN
-F 1 "R" V 2100 4500 50  0000 C CNN
+F 1 "10k" V 2100 4500 50  0000 C CNN
 F 2 "Resistor_THT:R_Axial_DIN0207_L6.3mm_D2.5mm_P10.16mm_Horizontal" V 1930 4400 50  0001 C CNN
 F 3 "~" H 2000 4400 50  0001 C CNN
@@
 P 2000 4700
 F 0 "R4" V 2100 4650 50  0000 C CNN
-F 1 "R" V 2100 4800 50  0000 C CNN
+F 1 "10k" V 2100 4800 50  0000 C CNN
 F 2 "Resistor_THT:R_Axial_DIN0207_L6.3mm_D2.5mm_P10.16mm_Horizontal" V 1930 4700 50  0001 C CNN
 F 3 "~" H 2000 4700 50  0001 C CNN
@@
 P 2000 2350
 F 0 "R1" V 2100 2300 50  0000 C CNN
-F 1 "R" V 2100 2450 50  0000 C CNN
+F 1 "10k" V 2100 2450 50  0000 C CNN
 F 2 "Resistor_THT:R_Axial_DIN0207_L6.3mm_D2.5mm_P10.16mm_Horizontal" V 1930 2350 50  0001 C CNN
 F 3 "~" H 2000 2350 50  0001 C CNN
@@
 P 2000 2650
 F 0 "R2" V 2100 2600 50  0000 C CNN
-F 1 "R" V 2100 2750 50  0000 C CNN
+F 1 "10k" V 2100 2750 50  0000 C CNN
 F 2 "Resistor_THT:R_Axial_DIN0207_L6.3mm_D2.5mm_P10.16mm_Horizontal" V 1930 2650 50  0001 C CNN
 F 3 "~" H 2000 2650 50  0001 C CNN
@@
 P 7650 2800
 F 0 "R21" V 7750 2750 50  0000 C CNN
-F 1 "R" V 7750 2900 50  0000 C CNN
+F 1 "10k" V 7750 2900 50  0000 C CNN
 F 2 "Resistor_THT:R_Axial_DIN0207_L6.3mm_D2.5mm_P10.16mm_Horizontal" V 7580 2800 50  0001 C CNN
 F 3 "~" H 7650 2800 50  0001 C CNN
@@
 P 7850 2800
 F 0 "R22" V 7950 2750 50  0000 C CNN
-F 1 "R" V 7950 2900 50  0000 C CNN
+F 1 "10k" V 7950 2900 50  0000 C CNN
 F 2 "Resistor_THT:R_Axial_DIN0207_L6.3mm_D2.5mm_P10.16mm_Horizontal" V 7780 2800 50  0001 C CNN
 F 3 "~" H 7850 2800 50  0001 C CNN
@@
 P 3300 2050
 F 0 "R5" V 3400 2000 50  0000 C CNN
-F 1 "R" V 3400 2150 50  0000 C CNN
+F 1 "680R" V 3400 2150 50  0000 C CNN
 F 2 "Resistor_THT:R_Axial_DIN0207_L6.3mm_D2.5mm_P10.16mm_Horizontal" V 3230 2050 50  0001 C CNN
 F 3 "~" H 3300 2050 50  0001 C CNN
@@
 P 3300 2150
 F 0 "R6" V 3400 2100 50  0000 C CNN
-F 1 "R" V 3400 2250 50  0000 C CNN
+F 1 "680R" V 3400 2250 50  0000 C CNN
 F 2 "Resistor_THT:R_Axial_DIN0207_L6.3mm_D2.5mm_P10.16mm_Horizontal" V 3230 2150 50  0001 C CNN
 F 3 "~" H 3300 2150 50  0001 C CNN
@@
 P 3300 2250
 F 0 "R7" V 3400 2200 50  0000 C CNN
-F 1 "R" V 3400 2350 50  0000 C CNN
+F 1 "680R" V 3400 2350 50  0000 C CNN
 F 2 "Resistor_THT:R_Axial_DIN0207_L6.3mm_D2.5mm_P10.16mm_Horizontal" V 3230 2250 50  0001 C CNN
 F 3 "~" H 3300 2250 50  0001 C CNN
@@
 P 3300 2350
 F 0 "R8" V 3400 2300 50  0000 C CNN
-F 1 "R" V 3400 2450 50  0000 C CNN
+F 1 "680R" V 3400 2450 50  0000 C CNN
 F 2 "Resistor_THT:R_Axial_DIN0207_L6.3mm_D2.5mm_P10.16mm_Horizontal" V 3230 2350 50  0001 C CNN
 F 3 "~" H 3300 2350 50  0001 C CNN
@@
 P 3300 2450
 F 0 "R9" V 3400 2400 50  0000 C CNN
-F 1 "R" V 3400 2550 50  0000 C CNN
+F 1 "680R" V 3400 2550 50  0000 C CNN
 F 2 "Resistor_THT:R_Axial_DIN0207_L6.3mm_D2.5mm_P10.16mm_Horizontal" V 3230 2450 50  0001 C CNN
 F 3 "~" H 3300 2450 50  0001 C CNN
@@
 P 3300 2550
 F 0 "R10" V 3400 2500 50  0000 C CNN
-F 1 "R" V 3400 2650 50  0000 C CNN
+F 1 "680R" V 3400 2650 50  0000 C CNN
 F 2 "Resistor_THT:R_Axial_DIN0207_L6.3mm_D2.5mm_P10.16mm_Horizontal" V 3230 2550 50  0001 C CNN
 F 3 "~" H 3300 2550 50  0001 C CNN
@@
 P 3300 2650
 F 0 "R11" V 3400 2600 50  0000 C CNN
-F 1 "R" V 3400 2750 50  0000 C CNN
+F 1 "680R" V 3400 2750 50  0000 C CNN
 F 2 "Resistor_THT:R_Axial_DIN0207_L6.3mm_D2.5mm_P10.16mm_Horizontal" V 3230 2650 50  0001 C CNN
 F 3 "~" H 3300 2650 50  0001 C CNN
@@
 P 3300 2750
 F 0 "R12" V 3400 2700 50  0000 C CNN
-F 1 "R" V 3400 2850 50  0000 C CNN
+F 1 "680R" V 3400 2850 50  0000 C CNN
 F 2 "Resistor_THT:R_Axial_DIN0207_L6.3mm_D2.5mm_P10.16mm_Horizontal" V 3230 2750 50  0001 C CNN
 F 3 "~" H 3300 2750 50  0001 C CNN
@@
 P 3300 4100
 F 0 "R13" V 3400 4050 50  0000 C CNN
-F 1 "R" V 3400 4200 50  0000 C CNN
+F 1 "680R" V 3400 4200 50  0000 C CNN
 F 2 "Resistor_THT:R_Axial_DIN0207_L6.3mm_D2.5mm_P10.16mm_Horizontal" V 3230 4100 50  0001 C CNN
 F 3 "~" H 3300 4100 50  0001 C CNN
@@
 P 3300 4200
 F 0 "R14" V 3400 4150 50  0000 C CNN
-F 1 "R" V 3400 4300 50  0000 C CNN
+F 1 "680R" V 3400 4300 50  0000 C CNN
 F 2 "Resistor_THT:R_Axial_DIN0207_L6.3mm_D2.5mm_P10.16mm_Horizontal" V 3230 4200 50  0001 C CNN
 F 3 "~" H 3300 4200 50  0001 C CNN
@@
 P 3300 4300
 F 0 "R15" V 3400 4250 50  0000 C CNN
-F 1 "R" V 3400 4400 50  0000 C CNN
+F 1 "220R" V 3400 4400 50  0000 C CNN
 F 2 "Resistor_THT:R_Axial_DIN0207_L6.3mm_D2.5mm_P10.16mm_Horizontal" V 3230 4300 50  0001 C CNN
 F 3 "~" H 3300 4300 50  0001 C CNN
@@
 P 3300 4400
 F 0 "R16" V 3400 4350 50  0000 C CNN
-F 1 "R" V 3400 4500 50  0000 C CNN
+F 1 "680R" V 3400 4500 50  0000 C CNN
 F 2 "Resistor_THT:R_Axial_DIN0207_L6.3mm_D2.5mm_P10.16mm_Horizontal" V 3230 4400 50  0001 C CNN
 F 3 "~" H 3300 4400 50  0001 C CNN
@@
 P 3300 4500
 F 0 "R17" V 3400 4450 50  0000 C CNN
-F 1 "R" V 3400 4600 50  0000 C CNN
+F 1 "220R" V 3400 4600 50  0000 C CNN
 F 2 "Resistor_THT:R_Axial_DIN0207_L6.3mm_D2.5mm_P10.16mm_Horizontal" V 3230 4500 50  0001 C CNN
 F 3 "~" H 3300 4500 50  0001 C CNN
@@
 P 3300 4600
 F 0 "R18" V 3400 4550 50  0000 C CNN
-F 1 "R" V 3400 4700 50  0000 C CNN
+F 1 "220R" V 3400 4700 50  0000 C CNN
 F 2 "Resistor_THT:R_Axial_DIN0207_L6.3mm_D2.5mm_P10.16mm_Horizontal" V 3230 4600 50  0001 C CNN
 F 3 "~" H 3300 4600 50  0001 C CNN
@@
 P 3300 4700
 F 0 "R19" V 3400 4650 50  0000 C CNN
-F 1 "R" V 3400 4800 50  0000 C CNN
+F 1 "220R" V 3400 4800 50  0000 C CNN
 F 2 "Resistor_THT:R_Axial_DIN0207_L6.3mm_D2.5mm_P10.16mm_Horizontal" V 3230 4700 50  0001 C CNN
 F 3 "~" H 3300 4700 50  0001 C CNN
@@
 P 3300 4800
 F 0 "R20" V 3400 4750 50  0000 C CNN
-F 1 "R" V 3400 4900 50  0000 C CNN
+F 1 "680R" V 3400 4900 50  0000 C CNN
 F 2 "Resistor_THT:R_Axial_DIN0207_L6.3mm_D2.5mm_P10.16mm_Horizontal" V 3230 4800 50  0001 C CNN
 F 3 "~" H 3300 4800 50  0001 C CNN
@@
 P 8600 1300
 F 0 "R23" V 8700 1250 50  0000 C CNN
-F 1 "R" V 8700 1400 50  0000 C CNN
+F 1 "1k" V 8700 1400 50  0000 C CNN
 F 2 "Resistor_THT:R_Axial_DIN0207_L6.3mm_D2.5mm_P10.16mm_Horizontal" V 8530 1300 50  0001 C CNN
 F 3 "~" H 8600 1300 50  0001 C CNN
@@
 P 8600 1700
 F 0 "R24" V 8700 1650 50  0000 C CNN
-F 1 "R" V 8700 1800 50  0000 C CNN
+F 1 "3.3k" V 8700 1800 50  0000 C CNN
 F 2 "Resistor_THT:R_Axial_DIN0207_L6.3mm_D2.5mm_P10.16mm_Horizontal" V 8530 1700 50  0001 C CNN
 F 3 "~" H 8600 1700 50  0001 C CNN
@@
 P 4300 4300
 F 0 "J9" H 4380 4292 50  0000 L CNN
-F 1 "Conn_SP_LED" H 4380 4201 50  0000 L CNN
+F 1 "Conn_MQTT_ERR" H 4380 4201 50  0000 L CNN
 F 2 "Connector_PinHeader_2.54mm:PinHeader_1x02_P2.54mm_Vertical" H 4300 4300 50  0001 C CNN
 F 3 "~" H 4300 4300 50  0001 C CNN
@@
 P 4300 4600
 F 0 "J10" H 4380 4592 50  0000 L CNN
-F 1 "Conn_Knob_LED" H 4380 4501 50  0000 L CNN
+F 1 "Conn_IP_LED" H 4380 4501 50  0000 L CNN
 F 2 "Connector_PinHeader_2.54mm:PinHeader_1x02_P2.54mm_Vertical" H 4300 4600 50  0001 C CNN
 F 3 "~" H 4300 4600 50  0001 C CNN
@@
 P 4300 4900
 F 0 "J11" H 4380 4892 50  0000 L CNN
-F 1 "Conn_IP_LED" H 4380 4801 50  0000 L CNN
+F 1 "Conn_Net_ERR" H 4380 4801 50  0000 L CNN
 F 2 "Connector_PinHeader_2.54mm:PinHeader_1x02_P2.54mm_Vertical" H 4300 4900 50  0001 C CNN
 F 3 "~" H 4300 4900 50  0001 C CNN
@@
 P 4300 5200
 F 0 "J12" H 4380 5192 50  0000 L CNN
-F 1 "Conn_Cloud_ERR" H 4380 5101 50  0000 L CNN
+F 1 "Conn_Knob_LED" H 4380 5101 50  0000 L CNN
 F 2 "Connector_PinHeader_2.54mm:PinHeader_1x02_P2.54mm_Vertical" H 4300 5200 50  0001 C CNN
 F 3 "~" H 4300 5200 50  0001 C CNN
@@
 P 4300 5500
 F 0 "J13" H 4380 5492 50  0000 L CNN
-F 1 "Conn_Network_ERR" H 4380 5401 50  0000 L CNN
+F 1 "Conn_Peri_ERR" H 4380 5401 50  0000 L CNN
 F 2 "Connector_PinHeader_2.54mm:PinHeader_1x02_P2.54mm_Vertical" H 4300 5500 50  0001 C CNN
 F 3 "~" H 4300 5500 50  0001 C CNN
@@
 P 4300 5800
 F 0 "J14" H 4380 5792 50  0000 L CNN
-F 1 "Conn_MQTT_ERR" H 4380 5701 50  0000 L CNN
+F 1 "Conn_SP_LED" H 4380 5701 50  0000 L CNN
 F 2 "Connector_PinHeader_2.54mm:PinHeader_1x02_P2.54mm_Vertical" H 4300 5800 50  0001 C CNN
 F 3 "~" H 4300 5800 50  0001 C CNN
@@
 P 10200 1700
 F 0 "R26" V 10300 1650 50  0000 C CNN
-F 1 "R" V 10300 1800 50  0000 C CNN
+F 1 "4.7k" V 10300 1800 50  0000 C CNN
 F 2 "Resistor_THT:R_Axial_DIN0207_L6.3mm_D2.5mm_P10.16mm_Horizontal" V 10130 1700 50  0001 C CNN
 F 3 "~" H 10200 1700 50  0001 C CNN
@@
 P 9950 1700
 F 0 "R25" V 10050 1650 50  0000 C CNN
-F 1 "R" V 10050 1800 50  0000 C CNN
+F 1 "4.7k" V 10050 1800 50  0000 C CNN
 F 2 "Resistor_THT:R_Axial_DIN0207_L6.3mm_D2.5mm_P10.16mm_Horizontal" V 9880 1700 50  0001 C CNN
 F 3 "~" H 9950 1700 50  0001 C CNN
